File: SingleCharger/SingleCharger.kicad_pcb (KiCad board)
At the start: 2 copper layers, 120 x 130 mm, 72 parts, among them J1 Bus_PCI_Express_x1, Q1 TPHR8504PL,LQ(M1W, Q2 TPHR8504PL,LQ(M1W, Q3 L2N7002SLLT1G, U1 ADS1115IDGSR, U10 LM358, U11 MCP4725A0T-E/CH, U12 MCP4725A0T-E/CH, U2 PICO, U3 TPS54360BDDAR, U4 TPS54360BDDAR, U5 NCP1117ST33T3G, U8 UCC27324DR, U9 LM393

Commit message: wORKING ON REFACTOR
Parts:
- removed C20, C21: 100n, Resistor_SMD:R_1206_3216Metric_Pad1.30x1.75mm_HandSolder
- removed D3, D4: D, Diode_SMD:D_1206_3216Metric_Pad1.42x1.75mm_HandSolder
- removed Q1: TPHR8504PL,LQ(M1W, COMPONENTS:DFN-5_L4.9-W5.9-P1.27-LS6.2-BL
- removed Q3: L2N7002SLLT1G, COMPONENTS:SOT-23-3_L3.0-W1.7-P0.95-LS2.9-BR
- removed R1: 0.003, Resistor_SMD:R_1206_3216Metric_Pad1.30x1.75mm_HandSolder
- removed R11: 100k, Resistor_SMD:R_1206_3216Metric_Pad1.30x1.75mm_HandSolder
- removed R13, R24, R25: 1k, Resistor_SMD:R_1206_3216Metric_Pad1.30x1.75mm_HandSolder
- removed R5, R9: 10k, Resistor_SMD:R_1206_3216Metric_Pad1.30x1.75mm_HandSolder
- removed U12: MCP4725A0T-E/CH, COMPONENTS:SOT-23-6_L2.9-W1.6-P0.95-LS2.8-BL
- added C23: 100n, Resistor_SMD:R_1206_3216Metric_Pad1.30x1.75mm_HandSolder, F.Cu at (94.7, 58.7)
- added C24: 100n, Resistor_SMD:R_1206_3216Metric_Pad1.30x1.75mm_HandSolder, F.Cu at (91.4, 77.0)
- C15, C16, Q2, R10, R2, U5, U9: moved to F.Cu
- moved C17 58.3 mm to (119.4, 51.1), turned to -90 degrees
- moved U1 40.6 mm to (113.3, 49.5), turned to -90 degrees
- moved R22 36.1 mm to (92.5, 70.1), turned to 90 degrees
- moved U11 35.9 mm to (75.9, 74.7), turned to 180 degrees
- moved C22 34.3 mm to (91.4, 80.0)
- moved U8 31.2 mm to (87.4, 85.3), turned to 0 degrees
- moved U9 25.8 mm to (86.1, 74.2), turned to 180 degrees
- moved R23 24.3 mm to (80.8, 75.4), turned to 90 degrees
- moved R3 23.2 mm to (68.4, 102.6)
- moved R4 23.2 mm to (68.4, 97.2)
- moved C19 19.9 mm to (77.0, 69.6), turned to -90 degrees
- moved C18 18.0 mm to (71.6, 73.7), turned to 180 degrees
- moved U5 17.8 mm to (75.2, 57.5), turned to -90 degrees
- moved R2 15.6 mm to (107.9, 68.9), turned to 90 degrees
- moved U10 15.6 mm to (96.5, 65.8), turned to 0 degrees
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Connections:
- C17 pad 2: /BatteryCC/3v3GND -> GND
- J1 pad A1: /BatteryCC/3v3GND -> GND
- Q2 pad 5: Net-(D3-K) -> /BatteryCC/B-
- U1 pad 1: /BatteryCC/3v3GND -> GND
- U1 pad 3: /BatteryCC/3v3GND -> GND
- U1 pad 7: /BatteryCC/RSns Discharge -> unconnected-(U1-AIN3-Pad7)
- U10 pad 5: Net-(Q1-D) -> unconnected-(U10B-+-Pad5)
- U10 pad 6: Net-(U10B--) -> unconnected-(U10B---Pad6)
- U10 pad 7: Net-(R11-Pad1) -> unconnected-(U10-Pad7)
- U2 pad 10: /BatteryCC/DischargeLV -> /DischargeLV
- U2 pad 6: /BatteryCC/En3v -> /En3v
- U8 pad 2: /BatteryCC/DischargeLV -> unconnected-(U8-INA-Pad2)
- U8 pad 7: Net-(U8-OUTA) -> unconnected-(U8-OUTA-Pad7)
- U9 pad 1: /BatteryCC/Discharge -> unconnected-(U9-Pad1)
- U9 pad 2: /BatteryCC/RSns Discharge -> unconnected-(U9A---Pad2)
- U9 pad 3: Net-(U9A-+) -> unconnected-(U9A-+-Pad3)
Routing:
- net /SDA: track 174.0 -> 28.7 mm, vias 7 -> 1
- net /SCL: track 169.6 -> 28.1 mm, vias 6 -> 1
- net /BatteryCC/En3v: track 139.3 -> 0.00 mm, vias 5 -> 0
- net /BatteryCC/Battery/EEPROM_WC: track 144.2 -> 27.5 mm, vias 3 -> 1
- net +5V: track 190.3 -> 100.0 mm, vias 3 -> 2
- net /BatteryCC/DischargeLV: track 85.6 -> 0.00 mm, vias 3 -> 0
- net +12V: track 105.1 -> 38.8 mm, vias 5 -> 3
- net /BatteryCC/ChargeLV: track 92.5 -> 26.4 mm, vias 3 -> 1
- net +3V3: track 99.4 -> 52.1 mm, vias 6 -> 0
- net /BatteryCC/RSns Discharge: track 42.5 -> 0.00 mm, vias 3 -> 0
- net /BatteryCC/B-: track 31.1 -> 0.00 mm, vias 3 -> 0
- net /BatteryCC/RSns Charge: track 35.6 -> 6.53 mm, vias 2 -> 0
- net /DischargeLV: track 0.00 -> 25.9 mm, vias 0 -> 1
- net GND: track 46.3 -> 22.2 mm, vias 297 -> 7
- net +24V: track 23.7 -> 1.87 mm, vias 1 -> 0
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- removed copper zone on B.Cu, net /BatteryCC/B-
- removed copper zone on B.Cu, net Net-(D3-K)
- removed copper zone on B.Cu, net Net-(D4-A)
- removed copper zone on B.Cu, net Net-(Q1-D)
- removed copper zone on B.Cu, net Net-(U10A-+)
Other:
- board text removed: "RSNS DSCHG"

Commit message: Added.
Parts:
- moved R3 63.6 mm to (130.3, 88.2)
- moved R4 63.6 mm to (130.3, 82.8)
- moved U1 7.52 mm to (111.8, 56.9), turned to 0 degrees
- moved C17 6.10 mm to (113.3, 50.8), turned to 0 degrees
- moved R20 4.67 mm to (102.9, 44.2), turned to 180 degrees
- moved R21 1.70 mm to (102.9, 46.7), turned to 180 degrees
Routing:
- net /SDA: track 28.7 -> 103.5 mm, vias 1 -> 3
- net /SCL: track 28.1 -> 99.8 mm
- net /BatteryCC/ChargeLV: track 26.4 -> 88.3 mm
- net +12V: track 38.8 -> 99.3 mm, vias 3 -> 5
- net /BatteryCC/ALERT/RDY: track 0.00 -> 55.8 mm, vias 0 -> 1
- net +3V3: track 52.1 -> 90.3 mm
- net /BatteryCC/Battery/EEPROM_WC: track 27.5 -> 0.50 mm, vias 1 -> 0
- net /DischargeLV: track 25.9 -> 0.00 mm, vias 1 -> 0
- net /BatteryCC/RSns Charge: track 6.53 -> 31.1 mm

Commit message: Working.
Parts:
- removed C15, C16: 10u, Capacitor_SMD:C_1206_3216Metric
- removed U5: NCP1117ST33T3G, COMPONENTS:SOT-223-3_L6.5-W3.4-P2.30-LS7.0-BR
- added R24: 1k, Resistor_SMD:R_1206_3216Metric_Pad1.30x1.75mm_HandSolder, B.Cu at (115.5, 117.6)
- added R25: 1k, Resistor_SMD:R_1206_3216Metric_Pad1.30x1.75mm_HandSolder, B.Cu at (115.5, 120.7)
- C1, C10, C11, C12, C13, C14, C17, C18, C19, C2, C22, C23, C24, C3, C4, C5, C6, C7, C8, C9, D1, D2, L1, L2, Q2, R10, R12, R14, R15, R16, R17, R18, R19, R2, R22, R23, R3, R4, R6, R7, R8, U1, U10, U11, U3, U4, U8, U9: moved to B.Cu
- moved R15 101.2 mm to (116.8, 52.0)
- moved R8 101.2 mm to (116.8, 47.0)
- moved L1 98.8 mm to (118.8, 33.6)
- moved C4 93.8 mm to (123.4, 46.2)
- moved R7 92.5 mm to (124.7, 50.0), turned to 180 degrees
- moved C5 91.0 mm to (126.2, 46.3)
- moved C6 90.8 mm to (126.4, 31.7)
- moved U2 89.2 mm to (102.0, 28.1), turned to 180 degrees
- moved C7 88.1 mm to (129.5, 31.7)
- moved D1 87.8 mm to (129.9, 38.3), turned to 0 degrees
- moved C23 85.5 mm to (143.8, 128.8), turned to 0 degrees
- moved C9 85.4 mm to (175.0, 95.0), turned to 0 degrees
- moved U3 85.2 mm to (133.3, 45.3)
- moved R6 83.5 mm to (136.1, 50.5)
- moved C3 82.1 mm to (138.9, 41.4)
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Connections:
- C17 pad 1: +3V3 -> +5V
- R12 pad 1: /BatteryCC/RSns Charge -> Net-(R12-Pad1)
- R22 pad 2: /BatteryCC/RSns Charge -> Net-(R12-Pad1)
- U1 pad 8: +3V3 -> +5V
- U10 pad 1: /BatteryCC/RSns Charge -> Net-(R12-Pad1)
- U2 pad 36: unconnected-(U2-3V3(OUT)-Pad36) -> +3V3
Routing:
- net /SCL: track 99.8 -> 3.24 mm, vias 1 -> 0
- net /SDA: track 103.5 -> 10.4 mm, vias 3 -> 0
- net /BatteryCC/ChargeLV: track 88.3 -> 0.00 mm, vias 1 -> 0
- net +3V3: track 90.3 -> 19.0 mm
- net /BatteryCC/ALERT/RDY: track 55.8 -> 0.00 mm, vias 1 -> 0
- net +5V: track 100.0 -> 62.1 mm
- net Net-(U1-AIN0): track 0.00 -> 33.1 mm
- net Net-(R12-Pad1): track 0.00 -> 26.6 mm
- net Net-(U10A-+): track 18.2 -> 32.4 mm
- net /BatteryCC/RSns Charge: track 31.1 -> 41.3 mm
- net /BatteryCC/Charge: track 23.4 -> 30.4 mm
- net +12V: track 99.3 -> 93.8 mm, vias 5 -> 8
- net /BatteryCC/B-: track 0.00 -> 5.10 mm
- net +24V: track 1.87 -> 5.79 mm
- net Net-(U8-OUTB): track 9.83 -> 13.6 mm
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- added copper zone on B.Cu, net +12V
- added copper zone on B.Cu, net +24V
- added copper zone on B.Cu, net +5V
- added copper zone on B.Cu, net Net-(D1-K)
- added copper zone on B.Cu, net Net-(D2-K)
- removed copper zone on F.Cu, net +12V
- removed copper zone on F.Cu, net +24V
- removed copper zone on F.Cu, net +5V
- removed copper zone on F.Cu, net Net-(D1-K)
- removed copper zone on F.Cu, net Net-(D2-K)
Other:
- board text removed: "+"
- board text removed: "-"
- board text removed: "0.003"
- board text removed: "100k"
- board text removed: "1k"
- board text removed: "3v3Reg"
- board text removed: "AMP"
- board text removed: "B+"
- board text removed: "B-"
- board text removed: "COMP"
- board text removed: "Charge Supply"
- board text removed: "GDRVE"
- board text removed: "PICO"
- board text removed: "RSNS CHG"
- board text removed: "VREF"

Commit message: Almost done with layout.
Parts:
- moved R3 19.3 mm to (138.9, 94.2), turned to 90 degrees
- moved R4 18.1 mm to (138.9, 89.2), turned to 90 degrees
- moved R10 15.1 mm to (142.7, 83.6)
- moved Q2 11.2 mm to (132.8, 79.6)
- moved R2 9.09 mm to (144.8, 79.0)
- moved U1 6.48 mm to (112.8, 82.0)
- moved J1 2.98 mm to (122.8, 89.9), turned to 0 degrees
- moved C17 2.40 mm to (102.9, 85.1), turned to -90 degrees
Routing:
- net +3V3: track 19.0 -> 148.6 mm, vias 0 -> 3
- net /BatteryCC/ChargeLV: track 0.00 -> 94.6 mm, vias 0 -> 1
- net /SDA: track 10.4 -> 102.5 mm, vias 0 -> 2
- net /SCL: track 3.24 -> 92.4 mm, vias 0 -> 3
- net +5V: track 62.1 -> 145.7 mm, vias 2 -> 4
- net /BatteryCC/Battery/EEPROM_WC: track 0.00 -> 60.3 mm, vias 0 -> 1
- net /BatteryCC/ALERT/RDY: track 0.00 -> 39.1 mm, vias 0 -> 1
- net /BatteryCC/Charge: track 30.4 -> 52.0 mm
- net Net-(U8-OUTB): track 13.6 -> 29.3 mm
- net Net-(U10A-+): track 32.4 -> 42.0 mm
- net /BatteryCC/RSns Charge: track 41.3 -> 49.4 mm, vias 0 -> 2
- net /BatteryCC/TMP: track 0.00 -> 7.43 mm
- net +24V: track 5.79 -> 7.67 mm
- net /BatteryCC/B-: track 5.10 -> 6.98 mm
- net Net-(U1-AIN0): track 33.1 -> 31.8 mm, vias 0 -> 2
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
Commit message: Finished layout and routing.
Routing:
- net GND: track 22.2 -> 27.5 mm, vias 1 -> 196
- net +3V3: track 148.6 -> 149.7 mm
- net /BatteryCC/Charge: track 52.0 -> 53.0 mm
- net +24V: track 7.67 -> 7.84 mm, vias 0 -> 12
- added copper zone on F.Cu, net +24V
- added copper zone on B.Cu, net /BatteryCC/B-
- added copper zone on B.Cu, net Net-(U10A-+)
Other:
- board text added: "0.003"
- board text added: "100K"
- board text added: "10K"
- board text added: "1K"
- board text added: "GDRIVE"
- board text added: "LM358"
- board text added: "V1.0"
